Commit message: updated the files from pakeage_gazebo, the model xacro and pluginds, works in ROS2 , the rest of the code idk

File: install/j8_xacro_model/share/j8_xacro_model/urdf/argo_j8.urdf.xacro (robot description, xacro)
@@ -9,7 +9,7 @@
   <xacro:property name="mesh_path" value="$(find j8_xacro_model)/meshes"/>
   <!-- Included Xacro Files -->
-  <xacro:include filename="$(find j8_xacro_model)/urdf/wheel.urdf.xacro"/>
+  <!-- <xacro:include filename="$(find j8_xacro_model)/urdf/wheel.urdf.xacro"/> -->
   <xacro:include filename="$(find j8_xacro_model)/urdf/set_color.xacro"/>
-  <xacro:include filename="$(find j8_xacro_model)/urdf/lidar.xacro"/>
+  <!-- <xacro:include filename="$(find j8_xacro_model)/urdf/lidar.xacro"/> -->
   <xacro:include filename="$(find j8_xacro_model)/urdf/panel.xacro"/>
   <xacro:include filename="$(find j8_xacro_model)/urdf/side_bar.xacro"/>
@@ -17,8 +17,5 @@
   <xacro:include filename="$(find j8_xacro_model)/urdf/gps.xacro"/>
   <xacro:include filename="$(find j8_xacro_model)/urdf/camera.xacro"/>
-  <!-- <xacro:include filename="$(find j8_xacro_model)/urdf/fixposition_holder.xacro"/>
-  <xacro:include filename="$(find j8_xacro_model)/urdf/fixposition_sensor.xacro"/> -->
   <xacro:include filename="$(find j8_xacro_model)/urdf/sick_lidar.urdf.xacro"/>
-  <xacro:include filename="$(find j8_xacro_model)/urdf/wheel.urdf.xacro"/>
   <xacro:include filename="$(find fixposition_sensor_pkg)/urdf/fixposition_main.xacro"/>
   <!--<xacro:include filename="$(find zed_camera_pkg)/urdf/camera_macro.urdf"/>-->
@@ -190,4 +187,112 @@
 <xacro:lidar name="velodyne" parent="J8_top" origin_xyz="1.6279 -0.0022244 0.17" origin_rpy="0 0 0" mass="0.61592" update_rate="10" min_angle="${-M_PI/2}" max_angle="${M_PI/2}" stddev="0.008" num_samples="431" min_range="0.2"  max_range="35.0" />
 <xacro:lidar name="sick" parent="J8_top" origin_xyz="1.50 0.02 0.27732" origin_rpy="0 0 0" mass="0.22144" update_rate="10" min_angle="${-M_PI/2}" max_angle="${M_PI/2}" stddev="0.008" num_samples="181" min_range="0.2"  max_range="8.0"/> -->
+    <link name="Sick_link">
+      <inertial>
+            <origin rpy="0 0 -1.5707963267948966" xyz="1.50 0.02 0.27732"/>
+            <mass value="0.22144"/>
+            <inertia ixx="0.00069055" ixy="0" ixz="0" iyy="0.0006838" iyz="0" izz="0.00083911"/>
+          </inertial>
+          <visual>
+            <origin rpy="0 0 0" xyz="0 0 0"/>
+            <geometry>
+              <mesh filename="file://$(find j8_xacro_model)/meshes/Sick.STL"/>
+            </geometry>
+            <!-- Default color for all lidars -->
+            <material name="">
+              <color rgba="0.5 0.5 0.5 1"/>
+            </material>
+          </visual>
+          <collision>
+            <origin rpy="0 0 0" xyz="0 0 0"/>
+            <geometry>
+              <mesh filename="file://$(find j8_xacro_model)/meshes/Sick.STL"/>
+            </geometry>
+          </collision>
+    </link>
+    <!-- Joint Definition -->
+    <joint name="Sick_joint" type="fixed">
+      <origin rpy="0 0 -1.5707963267948966" xyz="1.50 0.02 0.27732"/>
+      <parent link="J8_top"/>
+      <child link="Sick_link"/>
+      <axis xyz="0 0 0"/>
+    </joint>
+    <!-- Lidar -->
+  <link name="Velodyne_link">
+    <inertial>
+      <origin rpy="0 0 -1.5707963267948966" xyz="1.6279 -0.0022244 0.17"/>
+      <mass value="0.61592"/>
+      <inertia ixx="0.00069055" ixy="0" ixz="0" iyy="0.0006838" iyz="0" izz="0.00083911"/>
+    </inertial>
+    <visual>
+      <origin rpy="0 0 0" xyz="0 0 0"/>
+      <geometry>
+        <mesh filename="file://$(find j8_xacro_model)/meshes/Velodyne.STL"/>
+      </geometry>
+      <!-- Default color for all lidars -->
+      <material name="">
+        <color rgba="0.5 0.5 0.5 1"/>
+      </material>
+    </visual>
+    <collision>
+      <origin rpy="0 0 0" xyz="0 0 0"/>
+      <geometry>
+        <mesh filename="file://$(find j8_xacro_model)/meshes/Velodyne.STL"/>
+      </geometry>
+    </collision>
+  </link>
+  <joint name="Velodyne_joint" type="fixed">
+    <origin rpy="0 0 -1.5707963267948966" xyz="1.6279 -0.0022244 0.17"/>
+    <parent link="J8_top"/>
+    <child link="Velodyne_link"/>
+    <axis xyz="0 0 0"/>
+  </joint>
+  <gazebo reference="Velodyne_link">
+    <visual>
+      <material>
+        <ambient>0.8 0.8 0.8 1.0</ambient>
+        <diffuse>0.8 0.8 0.8 1.0</diffuse>
+        <specular>0.8 0.8 0.8 1.0</specular>
+        <emissive>0 0 0 0</emissive>
+      </material>
+    </visual>
+    <preserveFixedJoint>true</preserveFixedJoint>
+    <!-- Also preserve joint if has a fixed joint -->
+  </gazebo>
+<gazebo reference="Velodyne_link">
+    <sensor name="Velodyne" type="ray">
+      <pose>0 0 0 0 0 0</pose>
+      <visualize>1</visualize>
+      <update_rate>10</update_rate>
+      <ray>
+        <scan>
+          <horizontal>
+            <samples>431</samples>
+            <resolution>1</resolution>
+            <min_angle>0</min_angle>
+            <max_angle>3.141592653589793</max_angle>
+          </horizontal>
+        </scan>
+        <range>
+          <min>0.2</min>
+          <max>35.0</max>
+          <resolution>0.001</resolution>
+        </range>
+        <noise>
+          <type>gaussian</type>
+          <mean>0.0</mean>
+          <stddev>0.008</stddev>
+        </noise>
+      </ray>
+      <plugin filename="libgazebo_ros_ray_sensor.so" name="Velodyne_plugin">
+        <ros>
+          <namespace>ARGJ801</namespace>
+          <remapping>~/out:=/ARGJ801/Velodyne/scan</remapping>
+        </ros>
+        <!-- Fixed output type for all lidars -->
+        <output_type>sensor_msgs/LaserScan</output_type>
+        <frame_name>Velodyne_link</frame_name>
+      </plugin>
+    </sensor>
+  </gazebo>
 <!-- Front and Back Camera
 <xacro:camera name="Back_camera" parent="Bridge" origin_xyz="-0.11 0 0.18021" origin_rpy="0 1.5708 0" ros_topic="/back_camera"/>
@@ -204,4 +309,739 @@
 <xacro:wheel_with_suspension number="7" parent="base_link" suspension_xyz="0.32066 0.45 -0.225" wheel_xyz="0.0 0.18 0.0"/>
 <xacro:wheel_with_suspension number="8" parent="base_link" suspension_xyz="1.0107 0.45 -0.225" wheel_xyz="0.0 0.18 0.0"/> -->
+    <link name="Suspension_1">
+        <inertial>
+          <origin rpy="0 0 0" xyz="4.4409E-16 -0.005 2.2204E-16"/>
+          <mass value="10.0"/>
+          <inertia ixx="5.0" ixy="8.0515E-20" ixz="0" iyy="5.0" iyz="1.9328E-19" izz="5.0"/>
+        </inertial>
+        <visual>
+          <origin rpy="0 0 0" xyz="0 0 0"/>
+          <geometry>
+            <mesh filename="file://$(find j8_xacro_model)/meshes/Suspension_1.STL"/>
+          </geometry>
+          <material name="">
+            <color rgba="0.79216 0.81961 0.93333 1"/>
+          </material>
+        </visual>
+        <collision>
+          <origin rpy="0 0 0" xyz="0 0 0"/>
+          <geometry>
+            <mesh filename="file://$(find j8_xacro_model)/meshes/Suspension_1.STL"/>
+          </geometry>
+        </collision>
+    </link>
+      <!-- Prismatic Joint (Base Link to Suspension) -->
+      <joint name="base_Suspension_1_joint" type="prismatic">
+        <origin rpy=" 0 0 0 " xyz="-1.0593 -0.45 -0.225"/>
+        <parent link="base_link"/>
+        <child link="Suspension_1"/>
+        <axis xyz="0 0 1"/>
+        <limit effort="1000000000000.0" lower="-10.0" upper="10.0" velocity="0.0"/>
+        <dynamics damping="100.0" friction="1000000000000.0"/>
+      </joint>
+      <gazebo reference="base_Suspension_1_joint">
+        <implicitSpringDamper>true</implicitSpringDamper>
+        <springStiffness>500000000000000</springStiffness>
+        <springReference>0.0</springReference>
+      </gazebo>
+    <link name="Wheel_1">
+        <!-- Inertial, visual, and collision properties -->
+        <inertial>
+          <origin rpy="0 0 0" xyz="0 0.17637 0"/>
+          <mass value="5.205463824313"/>
+          <inertia ixx="3.66317923670982" ixy="0" ixz="0" iyy="3.66317923670982" iyz="0" izz="5.43484629444829"/>
+        </inertial>
+        <visual>
+          <origin rpy="1.5707963267948966 0 0" xyz="0 0 0"/>
+          <geometry>
+            <cylinder length="0.30" radius="0.298"/>
+          </geometry>
+          <geometry> <mesh filename="file://$(find j8_xacro_model)/meshes/Wheel1.STL"/>
+            </geometry>
+          <material name="">
+            <color rgba="0.792156862745098 0.819607843137255 0.933333333333333 1"/>
+          </material>
+        </visual>
+        <collision>
+          <origin rpy="1.5707963267948966 0 0" xyz="0 0 0"/>
+          <geometry>
+            <cylinder length="0.30" radius="0.298"/>
+          </geometry>
+          <geometry>
+              <mesh filename="file://$(find j8_xacro_model)/meshes/Wheel1.STL"/>
+            </geometry>
+        </collision>
+    </link>
+      <gazebo reference="Wheel_1">
+        <visual>
+          <material>
+            <ambient>0.0 0.0 0.0 1.0</ambient>
+            <diffuse>0.0 0.0 0.0 1.0</diffuse>
+            <specular>0.0 0.0 0.0 1.0</specular>
+            <emissive>0 0 0 0</emissive>
+          </material>
+        </visual>
+        <preserveFixedJoint>true</preserveFixedJoint>
+        <!-- Also preserve joint if has a fixed joint -->
+      </gazebo>
+      <gazebo reference="Wheel_1">
+        <kp>100000000000000.0</kp>
+        <kd>0.8</kd>
+        <mu>0.55</mu>
+        <mu2>0.55</mu2>
+        <fdir1> 1 0 0</fdir1>
+      </gazebo>
+      <joint name="Suspension_1_Wheel_1_joint" type="continuous">
+        <origin rpy="0 0 0" xyz="0.0 -0.18 0.0"/>
+        <parent link="Suspension_1"/>
+        <child link="Wheel_1"/>
+        <axis xyz="0 1 0"/>
+      </joint>
+      <gazebo reference="Suspension_1_Wheel_1_joint">
+      </gazebo>
+      <!-- Suspension Link -->
+      <link name="Suspension_2">
+        <inertial>
+          <origin rpy="0 0 0" xyz="4.4409E-16 -0.005 2.2204E-16"/>
+          <mass value="10.0"/>
+          <inertia ixx="5.0" ixy="8.0515E-20" ixz="0" iyy="5.0" iyz="1.9328E-19" izz="5.0"/>
+        </inertial>
+        <visual>
+          <origin rpy="0 0 0" xyz="0 0 0"/>
+          <geometry>
+            <mesh filename="file://$(find j8_xacro_model)/meshes/Suspension_2.STL"/>
+          </geometry>
+          <material name="">
+            <color rgba="0.79216 0.81961 0.93333 1"/>
+          </material>
+        </visual>
+        <collision>
+          <origin rpy="0 0 0" xyz="0 0 0"/>
+          <geometry>
+            <mesh filename="file://$(find j8_xacro_model)/meshes/Suspension_2.STL"/>
+          </geometry>
+        </collision>
+      </link>
+      <!-- Prismatic Joint (Base Link to Suspension) -->
+      <joint name="base_Suspension_2_joint" type="prismatic">
+        <origin rpy=" 0 0 0 " xyz="-0.36934 -0.45 -0.225"/>
+        <parent link="base_link"/>
+        <child link="Suspension_2"/>
+        <axis xyz="0 0 1"/>
+        <limit effort="1000000000000.0" lower="-10.0" upper="10.0" velocity="0.0"/>
+        <dynamics damping="100.0" friction="1000000000000.0"/>
+      </joint>
+      <gazebo reference="base_Suspension_2_joint">
+        <implicitSpringDamper>true</implicitSpringDamper>
+        <springStiffness>500000000000000</springStiffness>
+        <springReference>0.0</springReference>
+      </gazebo>
+      <link name="Wheel_2">
+        <!-- Inertial, visual, and collision properties -->
+        <inertial>
+          <origin rpy="0 0 0" xyz="0 0.17637 0"/>
+          <mass value="5.205463824313"/>
+          <inertia ixx="3.66317923670982" ixy="0" ixz="0" iyy="3.66317923670982" iyz="0" izz="5.43484629444829"/>
+        </inertial>
+        <visual>
+          <origin rpy="1.5707963267948966 0 0" xyz="0 0 0"/>
+          <geometry>
+            <cylinder length="0.30" radius="0.298"/>
+          </geometry>
+          <geometry> <mesh filename="file://$(find j8_xacro_model)/meshes/Wheel2.STL"/>
+            </geometry>
+          <material name="">
+            <color rgba="0.792156862745098 0.819607843137255 0.933333333333333 1"/>
+          </material>
+        </visual>
+        <collision>
+          <origin rpy="1.5707963267948966 0 0" xyz="0 0 0"/>
+          <geometry>
+            <cylinder length="0.30" radius="0.298"/>
+          </geometry>
+          <geometry>
+              <mesh filename="file://$(find j8_xacro_model)/meshes/Wheel2.STL"/>
+            </geometry>
+        </collision>
+      </link>
+      <gazebo reference="Wheel_2">
+        <visual>
+          <material>
+            <ambient>0.0 0.0 0.0 1.0</ambient>
+            <diffuse>0.0 0.0 0.0 1.0</diffuse>
+            <specular>0.0 0.0 0.0 1.0</specular>
+            <emissive>0 0 0 0</emissive>
+          </material>
+        </visual>
+        <preserveFixedJoint>true</preserveFixedJoint>
+        <!-- Also preserve joint if has a fixed joint -->
+      </gazebo>
+      <gazebo reference="Wheel_2">
+        <kp>100000000000000.0</kp>
+        <kd>0.8</kd>
+        <mu>0.55</mu>
+        <mu2>0.55</mu2>
+        <fdir1> 1 0 0</fdir1>
+      </gazebo>
+      <joint name="Suspension_2_Wheel_2_joint" type="continuous">
+        <origin rpy="0 0 0" xyz="0.0 -0.18 0.0"/>
+        <parent link="Suspension_2"/>
+        <child link="Wheel_2"/>
+        <axis xyz="0 1 0"/>
+      </joint>
+      <gazebo reference="Suspension_2_Wheel_2_joint">
+        </gazebo>
+      <!-- Suspension Link -->
+      <link name="Suspension_3">
+        <inertial>
+          <origin rpy="0 0 0" xyz="4.4409E-16 -0.005 2.2204E-16"/>
+          <mass value="10.0"/>
+          <inertia ixx="5.0" ixy="8.0515E-20" ixz="0" iyy="5.0" iyz="1.9328E-19" izz="5.0"/>
+        </inertial>
+        <visual>
+          <origin rpy="0 0 0" xyz="0 0 0"/>
+          <geometry>
+            <mesh filename="file://$(find j8_xacro_model)/meshes/Suspension_3.STL"/>
+          </geometry>
+          <material name="">
+            <color rgba="0.79216 0.81961 0.93333 1"/>
+          </material>
+        </visual>
+        <collision>
+          <origin rpy="0 0 0" xyz="0 0 0"/>
+          <geometry>
+            <mesh filename="file://$(find j8_xacro_model)/meshes/Suspension_3.STL"/>
+          </geometry>
+        </collision>
+      </link>
+      <!-- Prismatic Joint (Base Link to Suspension) -->
+      <joint name="base_Suspension_3_joint" type="prismatic">
+        <origin rpy=" 0 0 0 " xyz="0.32066 -0.45 -0.225"/>
+        <parent link="base_link"/>
+        <child link="Suspension_3"/>
+        <axis xyz="0 0 1"/>
+        <limit effort="1000000000000.0" lower="-10.0" upper="10.0" velocity="0.0"/>
+        <dynamics damping="100.0" friction="1000000000000.0"/>
+      </joint>
+      <gazebo reference="base_Suspension_3_joint">
+        <implicitSpringDamper>true</implicitSpringDamper>
+        <springStiffness>500000000000000</springStiffness>
+        <springReference>0.0</springReference>
+      </gazebo>
+      <link name="Wheel_3">
+        <!-- Inertial, visual, and collision properties -->
+        <inertial>
+          <origin rpy="0 0 0" xyz="0 0.17637 0"/>
+          <mass value="5.205463824313"/>
+          <inertia ixx="3.66317923670982" ixy="0" ixz="0" iyy="3.66317923670982" iyz="0" izz="5.43484629444829"/>
+        </inertial>
+        <visual>
+          <origin rpy="1.5707963267948966 0 0" xyz="0 0 0"/>
+          <geometry>
+            <cylinder length="0.30" radius="0.298"/>
+          </geometry>
+          <geometry> <mesh filename="file://$(find j8_xacro_model)/meshes/Wheel3.STL"/>
+            </geometry>
+          <material name="">
+            <color rgba="0.792156862745098 0.819607843137255 0.933333333333333 1"/>
+          </material>
+        </visual>
+        <collision>
+          <origin rpy="1.5707963267948966 0 0" xyz="0 0 0"/>
+          <geometry>
+            <cylinder length="0.30" radius="0.298"/>
+          </geometry>
+          <geometry>
+              <mesh filename="file://$(find j8_xacro_model)/meshes/Wheel3.STL"/>
+            </geometry>
+        </collision>
+      </link>
+      <gazebo reference="Wheel_3">
+        <visual>
+          <material>
+            <ambient>0.0 0.0 0.0 1.0</ambient>
+            <diffuse>0.0 0.0 0.0 1.0</diffuse>
+            <specular>0.0 0.0 0.0 1.0</specular>
+            <emissive>0 0 0 0</emissive>
+          </material>
+        </visual>
+        <preserveFixedJoint>true</preserveFixedJoint>
+        <!-- Also preserve joint if has a fixed joint -->
+      </gazebo>
+      <gazebo reference="Wheel_3">
+        <kp>100000000000000.0</kp>
+        <kd>0.8</kd>
+        <mu>0.55</mu>
+        <mu2>0.55</mu2>
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
File: install/j8_xacro_model/share/j8_xacro_model/urdf/lidar.xacro (robot description, xacro)
@@ -1,72 +1,39 @@
 <?xml version="1.0"?>
 <robot xmlns:xacro="http://www.ros.org/wiki/xacro">
-  <xacro:macro name="lidar" params="name parent origin_xyz origin_rpy mass update_rate min_angle max_angle stddev num_samples min_range max_range">
-    <link name="${name}_link">
-      <inertial>
-        <origin xyz="${origin_xyz}" rpy="${origin_rpy}" />
-        <mass value="${mass}" />
-        <inertia ixx="0.00069055" ixy="0" ixz="0" iyy="0.0006838" iyz="0" izz="0.00083911" />
-      </inertial>
-      <visual>
-        <origin xyz="0 0 0" rpy="0 0 0" />
-        <geometry>
-          <mesh filename="file://$(find j8_xacro_model)/meshes/${name}.STL" />
-        </geometry>
-        <!-- Default color for all lidars -->
-        <material name="">
-          <color rgba="0.5 0.5 0.5 1" />
-        </material>
-      </visual>
-      <collision>
-        <origin xyz="0 0 0" rpy="0 0 0" />
-        <geometry>
-          <mesh filename="file://$(find j8_xacro_model)/meshes/${name}.STL" />
-        </geometry>
-      </collision>
-    </link>
-    <joint name="${name}_joint" type="fixed">
-      <origin xyz="${origin_xyz}" rpy="${origin_rpy}" />
-      <parent link="${parent}" />
-      <child link="${name}_link" />
-      <axis xyz="0 0 0" />
-    </joint>
-   <xacro:set_gazebo_color link_name="${name}_link" r="0.8" g="0.8" b="0.8"/> <!-- Light Grey -->
-    <!-- Plugin Definition -->
-    <gazebo reference="${name}_link">
-      <sensor type="gpu_ray" name="${name}">
-        <pose>0 0 0 0 0 0</pose>
-        <visualize>1</visualize>
-        <update_rate>${update_rate}</update_rate>
-        <ray>
-          <scan>
-            <horizontal>
-              <samples>${num_samples}</samples>
-              <resolution>1</resolution>
-              <min_angle>${min_angle}</min_angle>
-              <max_angle>${max_angle}</max_angle>
-            </horizontal>
-          </scan>
-          <range>
-            <min>${min_range}</min>
-            <max>${max_range}</max>
-            <resolution>0.001</resolution>
-          </range>
-          <noise>
-            <type>gaussian</type>
-            <mean>0.0</mean>
-            <stddev>${stddev}</stddev>
-          </noise>
-        </ray>
-        <plugin name="${name}_plugin" filename="libgazebo_ros_ray_sensor.so">
-          <ros>
-            <namespace>${robot_namespace}</namespace>
-            <remapping>~/out:=/${robot_namespace}/${name}_scan</remapping>
-          </ros>
-          <!-- Fixed output type for all lidars -->
-          <output_type>sensor_msgs/LaserScan</output_type>
-          <frame_name>${name}_link</frame_name>
-        </plugin>
-      </sensor>
-    </gazebo>
-  </xacro:macro>
+ <gazebo reference="Velodyne_link">
+    <sensor name="Velodyne" type="ray">
+      <pose>0 0 0 0 0 0</pose>
+      <visualize>0</visualize>
+      <update_rate>10</update_rate>
+      <ray>
+        <scan>
+          <horizontal>
+            <samples>431</samples>
+            <resolution>1</resolution>
+            <min_angle>0</min_angle>
+            <max_angle>3.141592653589793</max_angle>
+          </horizontal>
+        </scan>
+        <range>
+          <min>0.2</min>
+          <max>35.0</max>
+          <resolution>0.001</resolution>
+        </range>
+        <noise>
+          <type>gaussian</type>
+          <mean>0.0</mean>
+          <stddev>0.008</stddev>
+        </noise>
+      </ray>
+      <plugin filename="libgazebo_ros_ray_sensor.so" name="Velodyne_plugin">
+        <ros>
+          <namespace>ARGJ801</namespace>
+          <remapping>~/out:=/ARGJ801/Velodyne/scan</remapping>
+        </ros>
+        <!-- Fixed output type for all lidars -->
+        <output_type>sensor_msgs/LaserScan</output_type>
+        <frame_name>Velodyne_link</frame_name>
+      </plugin>
+    </sensor>
+  </gazebo>
 </robot>

File: install/j8_xacro_model/share/j8_xacro_model/urdf/sick_lidar.urdf.xacro (robot description, xacro)
@@ -1,34 +1,4 @@
 <?xml version="1.0"?>
 <robot xmlns:xacro="http://www.ros.org/wiki/xacro">
-    <link name="Sick_link">
-      <inertial>
-            <origin rpy="0 0 -1.5707963267948966" xyz="1.50 0.02 0.27732"/>
-            <mass value="0.22144"/>
-            <inertia ixx="0.00069055" ixy="0" ixz="0" iyy="0.0006838" iyz="0" izz="0.00083911"/>
-          </inertial>
-          <visual>
-            <origin rpy="0 0 0" xyz="0 0 0"/>
-            <geometry>
-              <mesh filename="file://$(find j8_xacro_model)/meshes/Sick.STL"/>
-            </geometry>
-            <!-- Default color for all lidars -->
-            <material name="">
-              <color rgba="0.5 0.5 0.5 1"/>
-            </material>
-          </visual>
-          <collision>
-            <origin rpy="0 0 0" xyz="0 0 0"/>
-            <geometry>
-              <mesh filename="file://$(find j8_xacro_model)/meshes/Sick.STL"/>
-            </geometry>
-          </collision>
-    </link>
-    <!-- Joint Definition -->
-    <joint name="Sick_joint" type="fixed">
-      <origin rpy="0 0 -1.5707963267948966" xyz="1.50 0.02 0.27732"/>
-      <parent link="J8_top"/>
-      <child link="Sick_link"/>
-      <axis xyz="0 0 0"/>
-    </joint>
     <gazebo reference="Sick_link">
       <sensor type="gpu_ray" name="SickLidar">
@@ -56,8 +26,9 @@
           </noise>
         </ray>
-        <plugin name="lidar_controller" filename="libgazebo_ros_ray_sensor.so">
+        <plugin name="Sick_plugin" filename="libgazebo_ros_ray_sensor.so">
           <ros>
             <argument>use_sim_time:=true</argument>
-            <argument>~/out:=/sick_lidar</argument>
+            <namespace>ARGJ801</namespace>
+            <remapping>~/out:=/ARGJ801/Sick/scan</remapping>
           </ros>
           <frame_name>Sick_link</frame_name>
