Commit message: updated the files from pakeage_gazebo, the model xacro and pluginds, works in ROS2 , the rest of the code idk

File: install/j8_xacro_model/share/j8_xacro_model/urdf/wheel.urdf.xacro (robot description, xacro)
@@ -1,700 +1,75 @@
 <?xml version="1.0"?>
 <robot xmlns:xacro="http://www.ros.org/wiki/xacro">
-    <link name="Wheel_1">
-        <!-- Inertial, visual, and collision properties -->
-        <inertial>
-          <origin rpy="0 0 0" xyz="0 0.17637 0"/>
-          <mass value="5.205463824313"/>
-          <inertia ixx="3.66317923670982" ixy="0" ixz="0" iyy="3.66317923670982" iyz="0" izz="5.43484629444829"/>
-        </inertial>
-        <visual>
-          <origin rpy="1.5707963267948966 0 0" xyz="0 0 0"/>
-          <geometry>
-            <cylinder length="0.30" radius="0.298"/>
-          </geometry>
-          <!-- <geometry> <mesh filename="$(find j8_xacro_model)/meshes/${name}.STL"/>
-            </geometry>-->
-          <material name="">
-            <color rgba="0.792156862745098 0.819607843137255 0.933333333333333 1"/>
-          </material>
-        </visual>
-        <collision>
-          <origin rpy="1.5707963267948966 0 0" xyz="0 0 0"/>
-          <geometry>
-            <cylinder length="0.30" radius="0.298"/>
-          </geometry>
-          <!-- <geometry>
-              <mesh filename="$(find j8_xacro_model)/meshes/${name}.STL"/>
-            </geometry>-->
-        </collision>
-      </link>
-      <gazebo reference="Wheel_1">
-        <visual>
-          <material>
-            <ambient>0.0 0.0 0.0 1.0</ambient>
-            <diffuse>0.0 0.0 0.0 1.0</diffuse>
-            <specular>0.0 0.0 0.0 1.0</specular>
-            <emissive>0 0 0 0</emissive>
-          </material>
-        </visual>
-        <preserveFixedJoint>true</preserveFixedJoint>
-        <!-- Also preserve joint if has a fixed joint -->
-      </gazebo>
-      <gazebo reference="Wheel_1">
-        <kp>100000000000000.0</kp>
-        <kd>0.8</kd>
-        <mu>0.55</mu>
-        <mu2>0.55</mu2>
-        <fdir1> 1 0 0</fdir1>
-      </gazebo>
-      <joint name="Suspension_1_Wheel_1_joint" type="continuous">
-        <origin rpy="0 0 0" xyz="0.0 -0.18 0.0"/>
-        <parent link="Suspension_1"/>
-        <child link="Wheel_1"/>
-        <axis xyz="0 1 0"/>
-      </joint>
-      <gazebo reference="Suspension_1_Wheel_1_joint">
-        </gazebo>
-      <!-- Suspension Link -->
-      <link name="Suspension_2">
-        <inertial>
-          <origin rpy="0 0 0" xyz="4.4409E-16 -0.005 2.2204E-16"/>
-          <mass value="10.0"/>
-          <inertia ixx="5.0" ixy="8.0515E-20" ixz="0" iyy="5.0" iyz="1.9328E-19" izz="5.0"/>
-        </inertial>
-        <visual>
-          <origin rpy="0 0 0" xyz="0 0 0"/>
-          <geometry>
-            <mesh filename="/home/a/ARGOJ8_ws/install/j8_xacro_model/share/j8_xacro_model/meshes/Suspension_2.STL"/>
-          </geometry>
-          <material name="">
-            <color rgba="0.79216 0.81961 0.93333 1"/>
-          </material>
-        </visual>
-        <collision>
-          <origin rpy="0 0 0" xyz="0 0 0"/>
-          <geometry>
-            <mesh filename="/home/a/ARGOJ8_ws/install/j8_xacro_model/share/j8_xacro_model/meshes/Suspension_2.STL"/>
-          </geometry>
-        </collision>
-      </link>
-      <!-- Prismatic Joint (Base Link to Suspension) -->
-      <joint name="base_Suspension_2_joint" type="prismatic">
-        <origin rpy=" 0 0 0 " xyz="-0.36934 -0.45 -0.225"/>
-        <parent link="base_link"/>
-        <child link="Suspension_2"/>
-        <axis xyz="0 0 1"/>
-        <limit effort="1000000000000.0" lower="-10.0" upper="10.0" velocity="0.0"/>
-        <dynamics damping="100.0" friction="1000000000000.0"/>
-      </joint>
-      <gazebo reference="base_Suspension_2_joint">
-        <implicitSpringDamper>true</implicitSpringDamper>
-        <springStiffness>500000000000000</springStiffness>
-        <springReference>0.0</springReference>
-      </gazebo>
-      <link name="Wheel_2">
-        <!-- Inertial, visual, and collision properties -->
-        <inertial>
-          <origin rpy="0 0 0" xyz="0 0.17637 0"/>
-          <mass value="5.205463824313"/>
-          <inertia ixx="3.66317923670982" ixy="0" ixz="0" iyy="3.66317923670982" iyz="0" izz="5.43484629444829"/>
-        </inertial>
-        <visual>
-          <origin rpy="1.5707963267948966 0 0" xyz="0 0 0"/>
-          <geometry>
-            <cylinder length="0.30" radius="0.298"/>
-          </geometry>
-          <!-- <geometry> <mesh filename="$(find j8_xacro_model)/meshes/${name}.STL"/>
-            </geometry>-->
-          <material name="">
-            <color rgba="0.792156862745098 0.819607843137255 0.933333333333333 1"/>
-          </material>
-        </visual>
-        <collision>
-          <origin rpy="1.5707963267948966 0 0" xyz="0 0 0"/>
-          <geometry>
-            <cylinder length="0.30" radius="0.298"/>
-          </geometry>
-          <!-- <geometry>
-              <mesh filename="$(find j8_xacro_model)/meshes/${name}.STL"/>
-            </geometry>-->
-        </collision>
-      </link>
-      <gazebo reference="Wheel_2">
-        <visual>
-          <material>
-            <ambient>0.0 0.0 0.0 1.0</ambient>
-            <diffuse>0.0 0.0 0.0 1.0</diffuse>
-            <specular>0.0 0.0 0.0 1.0</specular>
-            <emissive>0 0 0 0</emissive>
-          </material>
-        </visual>
-        <preserveFixedJoint>true</preserveFixedJoint>
-        <!-- Also preserve joint if has a fixed joint -->
-      </gazebo>
-      <gazebo reference="Wheel_2">
-        <kp>100000000000000.0</kp>
-        <kd>0.8</kd>
-        <mu>0.55</mu>
-        <mu2>0.55</mu2>
-        <fdir1> 1 0 0</fdir1>
-      </gazebo>
-      <joint name="Suspension_2_Wheel_2_joint" type="continuous">
-        <origin rpy="0 0 0" xyz="0.0 -0.18 0.0"/>
-        <parent link="Suspension_2"/>
-        <child link="Wheel_2"/>
-        <axis xyz="0 1 0"/>
-      </joint>
-      <gazebo reference="Suspension_2_Wheel_2_joint">
-        </gazebo>
-      <!-- Suspension Link -->
-      <link name="Suspension_3">
-        <inertial>
-          <origin rpy="0 0 0" xyz="4.4409E-16 -0.005 2.2204E-16"/>
-          <mass value="10.0"/>
-          <inertia ixx="5.0" ixy="8.0515E-20" ixz="0" iyy="5.0" iyz="1.9328E-19" izz="5.0"/>
-        </inertial>
-        <visual>
-          <origin rpy="0 0 0" xyz="0 0 0"/>
-          <geometry>
-            <mesh filename="/home/a/ARGOJ8_ws/install/j8_xacro_model/share/j8_xacro_model/meshes/Suspension_3.STL"/>
-          </geometry>
-          <material name="">
-            <color rgba="0.79216 0.81961 0.93333 1"/>
-          </material>
-        </visual>
-        <collision>
-          <origin rpy="0 0 0" xyz="0 0 0"/>
-          <geometry>
-            <mesh filename="/home/a/ARGOJ8_ws/install/j8_xacro_model/share/j8_xacro_model/meshes/Suspension_3.STL"/>
-          </geometry>
-        </collision>
-      </link>
-      <!-- Prismatic Joint (Base Link to Suspension) -->
-      <joint name="base_Suspension_3_joint" type="prismatic">
-        <origin rpy=" 0 0 0 " xyz="0.32066 -0.45 -0.225"/>
-        <parent link="base_link"/>
-        <child link="Suspension_3"/>
-        <axis xyz="0 0 1"/>
-        <limit effort="1000000000000.0" lower="-10.0" upper="10.0" velocity="0.0"/>
-        <dynamics damping="100.0" friction="1000000000000.0"/>
-      </joint>
-      <gazebo reference="base_Suspension_3_joint">
-        <implicitSpringDamper>true</implicitSpringDamper>
-        <springStiffness>500000000000000</springStiffness>
-        <springReference>0.0</springReference>
-      </gazebo>
-      <link name="Wheel_3">
-        <!-- Inertial, visual, and collision properties -->
-        <inertial>
-          <origin rpy="0 0 0" xyz="0 0.17637 0"/>
-          <mass value="5.205463824313"/>
-          <inertia ixx="3.66317923670982" ixy="0" ixz="0" iyy="3.66317923670982" iyz="0" izz="5.43484629444829"/>
-        </inertial>
-        <visual>
-          <origin rpy="1.5707963267948966 0 0" xyz="0 0 0"/>
-          <geometry>
-            <cylinder length="0.30" radius="0.298"/>
-          </geometry>
-          <!-- <geometry> <mesh filename="$(find j8_xacro_model)/meshes/${name}.STL"/>
-            </geometry>-->
-          <material name="">
-            <color rgba="0.792156862745098 0.819607843137255 0.933333333333333 1"/>
-          </material>
-        </visual>
-        <collision>
-          <origin rpy="1.5707963267948966 0 0" xyz="0 0 0"/>
-          <geometry>
-            <cylinder length="0.30" radius="0.298"/>
-          </geometry>
-          <!-- <geometry>
-              <mesh filename="$(find j8_xacro_model)/meshes/${name}.STL"/>
-            </geometry>-->
-        </collision>
-      </link>
-      <gazebo reference="Wheel_3">
-        <visual>
-          <material>
-            <ambient>0.0 0.0 0.0 1.0</ambient>
-            <diffuse>0.0 0.0 0.0 1.0</diffuse>
-            <specular>0.0 0.0 0.0 1.0</specular>
-            <emissive>0 0 0 0</emissive>
-          </material>
-        </visual>
-        <preserveFixedJoint>true</preserveFixedJoint>
-        <!-- Also preserve joint if has a fixed joint -->
-      </gazebo>
-      <gazebo reference="Wheel_3">
-        <kp>100000000000000.0</kp>
-        <kd>0.8</kd>
-        <mu>0.55</mu>
-        <mu2>0.55</mu2>
-        <fdir1> 1 0 0</fdir1>
-      </gazebo>
-      <joint name="Suspension_3_Wheel_3_joint" type="continuous">
-        <origin rpy="0 0 0" xyz="0.0 -0.18 0.0"/>
-        <parent link="Suspension_3"/>
-        <child link="Wheel_3"/>
-        <axis xyz="0 1 0"/>
-      </joint>
-      <gazebo reference="Suspension_3_Wheel_3_joint">
-        </gazebo>
-      <!-- Suspension Link -->
-      <link name="Suspension_4">
-        <inertial>
-          <origin rpy="0 0 0" xyz="4.4409E-16 -0.005 2.2204E-16"/>
-          <mass value="10.0"/>
-          <inertia ixx="5.0" ixy="8.0515E-20" ixz="0" iyy="5.0" iyz="1.9328E-19" izz="5.0"/>
-        </inertial>
-        <visual>
-          <origin rpy="0 0 0" xyz="0 0 0"/>
-          <geometry>
-            <mesh filename="/home/a/ARGOJ8_ws/install/j8_xacro_model/share/j8_xacro_model/meshes/Suspension_4.STL"/>
-          </geometry>
-          <material name="">
-            <color rgba="0.79216 0.81961 0.93333 1"/>
-          </material>
-        </visual>
-        <collision>
-          <origin rpy="0 0 0" xyz="0 0 0"/>
-          <geometry>
-            <mesh filename="/home/a/ARGOJ8_ws/install/j8_xacro_model/share/j8_xacro_model/meshes/Suspension_4.STL"/>
-          </geometry>
-        </collision>
-      </link>
-      <!-- Prismatic Joint (Base Link to Suspension) -->
-      <joint name="base_Suspension_4_joint" type="prismatic">
-        <origin rpy=" 0 0 0 " xyz="1.0107 -0.45 -0.225"/>
-        <parent link="base_link"/>
-        <child link="Suspension_4"/>
-        <axis xyz="0 0 1"/>
-        <limit effort="1000000000000.0" lower="-10.0" upper="10.0" velocity="0.0"/>
-        <dynamics damping="100.0" friction="1000000000000.0"/>
-      </joint>
-      <gazebo reference="base_Suspension_4_joint">
-        <implicitSpringDamper>true</implicitSpringDamper>
-        <springStiffness>500000000000000</springStiffness>
-        <springReference>0.0</springReference>
-      </gazebo>
-      <link name="Wheel_4">
-        <!-- Inertial, visual, and collision properties -->
-        <inertial>
-          <origin rpy="0 0 0" xyz="0 0.17637 0"/>
-          <mass value="5.205463824313"/>
-          <inertia ixx="3.66317923670982" ixy="0" ixz="0" iyy="3.66317923670982" iyz="0" izz="5.43484629444829"/>
-        </inertial>
-        <visual>
-          <origin rpy="1.5707963267948966 0 0" xyz="0 0 0"/>
-          <geometry>
-            <cylinder length="0.30" radius="0.298"/>
-          </geometry>
-          <!-- <geometry> <mesh filename="$(find j8_xacro_model)/meshes/${name}.STL"/>
-            </geometry>-->
-          <material name="">
-            <color rgba="0.792156862745098 0.819607843137255 0.933333333333333 1"/>
-          </material>
-        </visual>
-        <collision>
-          <origin rpy="1.5707963267948966 0 0" xyz="0 0 0"/>
-          <geometry>
-            <cylinder length="0.30" radius="0.298"/>
-          </geometry>
-          <!-- <geometry>
-              <mesh filename="$(find j8_xacro_model)/meshes/${name}.STL"/>
-            </geometry>-->
-        </collision>
-      </link>
-      <gazebo reference="Wheel_4">
-        <visual>
-          <material>
-            <ambient>0.0 0.0 0.0 1.0</ambient>
-            <diffuse>0.0 0.0 0.0 1.0</diffuse>
-            <specular>0.0 0.0 0.0 1.0</specular>
-            <emissive>0 0 0 0</emissive>
-          </material>
-        </visual>
-        <preserveFixedJoint>true</preserveFixedJoint>
-        <!-- Also preserve joint if has a fixed joint -->
-      </gazebo>
-      <gazebo reference="Wheel_4">
-        <kp>100000000000000.0</kp>
-        <kd>0.8</kd>
-        <mu>0.55</mu>
-        <mu2>0.55</mu2>
-        <fdir1> 1 0 0</fdir1>
-      </gazebo>
-      <joint name="Suspension_4_Wheel_4_joint" type="continuous">
-        <origin rpy="0 0 0" xyz="0.0 -0.18 0.0"/>
-        <parent link="Suspension_4"/>
-        <child link="Wheel_4"/>
-        <axis xyz="0 1 0"/>
-      </joint>
-      <gazebo reference="Suspension_4_Wheel_4_joint">
-        </gazebo>
-      <!-- Suspension Link -->
-      <link name="Suspension_5">
-        <inertial>
-          <origin rpy="0 0 0" xyz="4.4409E-16 -0.005 2.2204E-16"/>
-          <mass value="10.0"/>
-          <inertia ixx="5.0" ixy="8.0515E-20" ixz="0" iyy="5.0" iyz="1.9328E-19" izz="5.0"/>
-        </inertial>
-        <visual>
-          <origin rpy="0 0 0" xyz="0 0 0"/>
-          <geometry>
-            <mesh filename="/home/a/ARGOJ8_ws/install/j8_xacro_model/share/j8_xacro_model/meshes/Suspension_5.STL"/>
-          </geometry>
-          <material name="">
-            <color rgba="0.79216 0.81961 0.93333 1"/>
-          </material>
-        </visual>
-        <collision>
-          <origin rpy="0 0 0" xyz="0 0 0"/>
-          <geometry>
-            <mesh filename="/home/a/ARGOJ8_ws/install/j8_xacro_model/share/j8_xacro_model/meshes/Suspension_5.STL"/>
-          </geometry>
-        </collision>
-      </link>
-      <!-- Prismatic Joint (Base Link to Suspension) -->
-      <joint name="base_Suspension_5_joint" type="prismatic">
-        <origin rpy=" 0 0 0 " xyz="-1.0593 0.45 -0.225"/>
-        <parent link="base_link"/>
-        <child link="Suspension_5"/>
-        <axis xyz="0 0 1"/>
-        <limit effort="1000000000000.0" lower="-10.0" upper="10.0" velocity="0.0"/>
-        <dynamics damping="100.0" friction="1000000000000.0"/>
-      </joint>
-      <gazebo reference="base_Suspension_5_joint">
-        <implicitSpringDamper>true</implicitSpringDamper>
-        <springStiffness>500000000000000</springStiffness>
-        <springReference>0.0</springReference>
-      </gazebo>
-      <link name="Wheel_5">
-        <!-- Inertial, visual, and collision properties -->
-        <inertial>
-          <origin rpy="0 0 0" xyz="0 0.17637 0"/>
-          <mass value="5.205463824313"/>
-          <inertia ixx="3.66317923670982" ixy="0" ixz="0" iyy="3.66317923670982" iyz="0" izz="5.43484629444829"/>
-        </inertial>
-        <visual>
-          <origin rpy="1.5707963267948966 0 0" xyz="0 0 0"/>
-          <geometry>
-            <cylinder length="0.30" radius="0.298"/>
-          </geometry>
-          <!-- <geometry> <mesh filename="$(find j8_xacro_model)/meshes/${name}.STL"/>
-            </geometry>-->
-          <material name="">
-            <color rgba="0.792156862745098 0.819607843137255 0.933333333333333 1"/>
-          </material>
-        </visual>
-        <collision>
-          <origin rpy="1.5707963267948966 0 0" xyz="0 0 0"/>
-          <geometry>
-            <cylinder length="0.30" radius="0.298"/>
-          </geometry>
-          <!-- <geometry>
-              <mesh filename="$(find j8_xacro_model)/meshes/${name}.STL"/>
-            </geometry>-->
-        </collision>
-      </link>
-      <gazebo reference="Wheel_5">
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