Commit message: update

File: install/j8_xacro_model/share/j8_xacro_model/urdf/argo_j8.xacro (robot description, xacro)
@@ -242,5 +242,5 @@
   </link>
   <joint name="Velodyne_joint" type="fixed">
-    <origin rpy="0 0 -1.5707963267948966" xyz="1.6279 -0.0022244 0.17"/>
+    <origin rpy="0 0 0" xyz="1.6279 -0.0022244 0.17"/>
     <parent link="J8_top"/>
     <child link="Velodyne_link"/>
