Commit message: added few launches

File: install/car/share/car/urdf/car.xacro (robot description, xacro)
@@ -531,5 +531,10 @@
   <child link="lidar_footprint"/>
   <!-- Ajusta rpy para alinear el frame óptico -->
-  <origin xyz="0 0 0" rpy="0 0 0"/>
+  <!--
+    Corrección de orientación:
+    Si la nube de puntos se ve girada +90° (hacia la izquierda visto desde el frente),
+    rotamos el frame del LiDAR -90° alrededor de Z.
+  -->
+  <origin xyz="0 0 0" rpy="0 0 -1.5708"/>
 </joint>
  <gazebo>

File: install/j8_xacro_model/share/j8_xacro_model/urdf/lidar.plugin.xacro (robot description, xacro)
@@ -39,5 +39,10 @@
           <remapping>~/out:=/ARGJ801/Velodyne/scan_cloud</remapping>
         </ros>
-        <!-- Fixed output type for all lidars -->
+        <!--
+          IMPORTANT:
+          Si publicamos la nube con frame_name=base_link, la nube se verá "girada" si
+          el link del sensor (Velodyne_link) tiene una orientación distinta en TF.
+          Publica con el frame del sensor para respetar el yaw/pitch/roll del joint.
+        -->
         <frame_name>Velodyne_link</frame_name>
         <output_type>sensor_msgs/PointCloud2</output_type>
