Commit message: update the code , refiene the control node, the rest need to refien the last thigns but works averall

File: src/gazebo_sim_pkgs/j8_xacro_model/urdf/argo_j8.xacro (robot description, xacro)
@@ -220,5 +220,5 @@
   <link name="Velodyne_link">
     <inertial>
-      <origin rpy="0 0 -1.5707963267948966" xyz="1.6279 -0.0022244 0.17"/>
+      <origin rpy="0 0 -1.5707963267948966" xyz="0.93 0.0 1.0"/>
       <mass value="0.61592"/>
       <inertia ixx="0.00069055" ixy="0" ixz="0" iyy="0.0006838" iyz="0" izz="0.00083911"/>
@@ -242,5 +242,5 @@
   </link>
   <joint name="Velodyne_joint" type="fixed">
-    <origin rpy="0 0 0" xyz="1.6279 -0.0022244 0.17"/>
+    <origin rpy="0 0 0" xyz="0.93 0.0 1.0"/>
     <parent link="J8_top"/>
     <child link="Velodyne_link"/>
