Commit message: update the code

File: src/gazebo_sim_pkgs/j8_xacro_model/urdf/argo_j8.xacro (robot description, xacro)
@@ -43,5 +43,5 @@
       <geometry>
         <mesh
-          filename="file://$(find j8_xacro_model)/meshes/base_link.STL" />
+          filename="package://j8_xacro_model/meshes/base_link.STL" />
       </geometry>
       <material
@@ -57,5 +57,5 @@
       <geometry>
         <mesh
-          filename="file://$(find j8_xacro_model)/meshes/base_link.STL" />
+          filename="package://j8_xacro_model/meshes/base_link.STL" />
       </geometry>
     </collision>
@@ -85,5 +85,5 @@
       <geometry>
         <mesh
-          filename="file://$(find j8_xacro_model)/meshes/J8_top.STL" />
+          filename="package://j8_xacro_model/meshes/J8_top.STL" />
       </geometry>
       <material
@@ -99,5 +99,5 @@
       <geometry>
         <mesh
-          filename="file://$(find j8_xacro_model)/meshes/J8_top.STL" />
+          filename="package://j8_xacro_model/meshes/J8_top.STL" />
       </geometry>
     </collision>
@@ -139,5 +139,5 @@
       <geometry>
         <mesh
-          filename="file://$(find j8_xacro_model)/meshes/Bridge.STL" />
+          filename="package://j8_xacro_model/meshes/Bridge.STL" />
       </geometry>
       <material
@@ -153,5 +153,5 @@
       <geometry>
         <mesh
-          filename="file://$(find j8_xacro_model)/meshes/Bridge.STL" />
+          filename="package://j8_xacro_model/meshes/Bridge.STL" />
       </geometry>
     </collision>
@@ -196,5 +196,5 @@
             <origin rpy="0 0 0" xyz="0 0 0"/>
             <geometry>
-              <mesh filename="file://$(find j8_xacro_model)/meshes/Sick.STL"/>
+              <mesh filename="package://j8_xacro_model/meshes/Sick.STL"/>
             </geometry>
             <!-- Default color for all lidars -->
@@ -206,5 +206,5 @@
             <origin rpy="0 0 0" xyz="0 0 0"/>
             <geometry>
-              <mesh filename="file://$(find j8_xacro_model)/meshes/Sick.STL"/>
+              <mesh filename="package://j8_xacro_model/meshes/Sick.STL"/>
             </geometry>
           </collision>
@@ -227,5 +227,5 @@
       <origin rpy="0 0 0" xyz="0 0 0"/>
       <geometry>
-        <mesh filename="file://$(find j8_xacro_model)/meshes/Velodyne.STL"/>
+        <mesh filename="package://j8_xacro_model/meshes/Velodyne.STL"/>
       </geometry>
       <!-- Default color for all lidars -->
@@ -237,5 +237,5 @@
       <origin rpy="0 0 0" xyz="0 0 0"/>
       <geometry>
-        <mesh filename="file://$(find j8_xacro_model)/meshes/Velodyne.STL"/>
+        <mesh filename="package://j8_xacro_model/meshes/Velodyne.STL"/>
       </geometry>
     </collision>
@@ -282,5 +282,5 @@
           <origin rpy="0 0 0" xyz="0 0 0"/>
           <geometry>
-            <mesh filename="file://$(find j8_xacro_model)/meshes/Suspension_1.STL"/>
+            <mesh filename="package://j8_xacro_model/meshes/Suspension_1.STL"/>
           </geometry>
           <material name="">
@@ -291,5 +291,5 @@
           <origin rpy="0 0 0" xyz="0 0 0"/>
           <geometry>
-            <mesh filename="file://$(find j8_xacro_model)/meshes/Suspension_1.STL"/>
+            <mesh filename="package://j8_xacro_model/meshes/Suspension_1.STL"/>
           </geometry>
         </collision>
@@ -321,5 +321,5 @@
             <cylinder length="0.30" radius="0.298"/>
           </geometry>
-          <geometry> <mesh filename="file://$(find j8_xacro_model)/meshes/Wheel1.STL"/>
+          <geometry> <mesh filename="package://j8_xacro_model/meshes/Wheel1.STL"/>
             </geometry>
           <material name="">
@@ -333,5 +333,5 @@
           </geometry>
           <geometry>
-              <mesh filename="file://$(find j8_xacro_model)/meshes/Wheel1.STL"/>
+              <mesh filename="package://j8_xacro_model/meshes/Wheel1.STL"/>
             </geometry>
         </collision>
@@ -374,5 +374,5 @@
           <origin rpy="0 0 0" xyz="0 0 0"/>
           <geometry>
-            <mesh filename="file://$(find j8_xacro_model)/meshes/Suspension_2.STL"/>
+            <mesh filename="package://j8_xacro_model/meshes/Suspension_2.STL"/>
           </geometry>
           <material name="">
@@ -383,5 +383,5 @@
           <origin rpy="0 0 0" xyz="0 0 0"/>
           <geometry>
-            <mesh filename="file://$(find j8_xacro_model)/meshes/Suspension_2.STL"/>
+            <mesh filename="package://j8_xacro_model/meshes/Suspension_2.STL"/>
           </geometry>
         </collision>
@@ -413,5 +413,5 @@
             <cylinder length="0.30" radius="0.298"/>
           </geometry>
-          <geometry> <mesh filename="file://$(find j8_xacro_model)/meshes/Wheel2.STL"/>
+          <geometry> <mesh filename="package://j8_xacro_model/meshes/Wheel2.STL"/>
             </geometry>
           <material name="">
@@ -425,5 +425,5 @@
           </geometry>
           <geometry>
-              <mesh filename="file://$(find j8_xacro_model)/meshes/Wheel2.STL"/>
+              <mesh filename="package://j8_xacro_model/meshes/Wheel2.STL"/>
             </geometry>
         </collision>
@@ -466,5 +466,5 @@
           <origin rpy="0 0 0" xyz="0 0 0"/>
           <geometry>
-            <mesh filename="file://$(find j8_xacro_model)/meshes/Suspension_3.STL"/>
+            <mesh filename="package://j8_xacro_model/meshes/Suspension_3.STL"/>
           </geometry>
           <material name="">
@@ -475,5 +475,5 @@
           <origin rpy="0 0 0" xyz="0 0 0"/>
           <geometry>
-            <mesh filename="file://$(find j8_xacro_model)/meshes/Suspension_3.STL"/>
+            <mesh filename="package://j8_xacro_model/meshes/Suspension_3.STL"/>
           </geometry>
         </collision>
@@ -505,5 +505,5 @@
             <cylinder length="0.30" radius="0.298"/>
           </geometry>
-          <geometry> <mesh filename="file://$(find j8_xacro_model)/meshes/Wheel3.STL"/>
+          <geometry> <mesh filename="package://j8_xacro_model/meshes/Wheel3.STL"/>
             </geometry>
           <material name="">
@@ -517,5 +517,5 @@
           </geometry>
           <geometry>
-              <mesh filename="file://$(find j8_xacro_model)/meshes/Wheel3.STL"/>
+              <mesh filename="package://j8_xacro_model/meshes/Wheel3.STL"/>
             </geometry>
         </collision>
@@ -558,5 +558,5 @@
           <origin rpy="0 0 0" xyz="0 0 0"/>
           <geometry>
-            <mesh filename="file://$(find j8_xacro_model)/meshes/Suspension_4.STL"/>
+            <mesh filename="package://j8_xacro_model/meshes/Suspension_4.STL"/>
           </geometry>
           <material name="">
@@ -567,5 +567,5 @@
           <origin rpy="0 0 0" xyz="0 0 0"/>
           <geometry>
-            <mesh filename="file://$(find j8_xacro_model)/meshes/Suspension_4.STL"/>
+            <mesh filename="package://j8_xacro_model/meshes/Suspension_4.STL"/>
           </geometry>
         </collision>
@@ -597,5 +597,5 @@
             <cylinder length="0.30" radius="0.298"/>
           </geometry>
-          <geometry> <mesh filename="file://$(find j8_xacro_model)/meshes/Wheel4.STL"/>
+          <geometry> <mesh filename="package://j8_xacro_model/meshes/Wheel4.STL"/>
             </geometry>
           <material name="">
@@ -609,5 +609,5 @@
           </geometry>
           <geometry>
-              <mesh filename="file://$(find j8_xacro_model)/meshes/Wheel4.STL"/>
+              <mesh filename="package://j8_xacro_model/meshes/Wheel4.STL"/>
             </geometry>
         </collision>
@@ -650,5 +650,5 @@
           <origin rpy="0 0 0" xyz="0 0 0"/>
           <geometry>
-            <mesh filename="file://$(find j8_xacro_model)/meshes/Suspension_5.STL"/>
+            <mesh filename="package://j8_xacro_model/meshes/Suspension_5.STL"/>
           </geometry>
           <material name="">
@@ -659,5 +659,5 @@
           <origin rpy="0 0 0" xyz="0 0 0"/>
           <geometry>
-            <mesh filename="file://$(find j8_xacro_model)/meshes/Suspension_5.STL"/>
+            <mesh filename="package://j8_xacro_model/meshes/Suspension_5.STL"/>
           </geometry>
         </collision>
@@ -689,5 +689,5 @@
             <cylinder length="0.30" radius="0.298"/>
           </geometry>
-          <geometry> <mesh filename="file://$(find j8_xacro_model)/meshes/Wheel5.STL"/>
+          <geometry> <mesh filename="package://j8_xacro_model/meshes/Wheel5.STL"/>
             </geometry>
           <material name="">
@@ -701,5 +701,5 @@
           </geometry>
           <geometry>
-              <mesh filename="file://$(find j8_xacro_model)/meshes/Wheel5.STL"/>
+              <mesh filename="package://j8_xacro_model/meshes/Wheel5.STL"/>
             </geometry>
         </collision>
@@ -742,5 +742,5 @@
           <origin rpy="0 0 0" xyz="0 0 0"/>
           <geometry>
-            <mesh filename="file://$(find j8_xacro_model)/meshes/Suspension_6.STL"/>
+            <mesh filename="package://j8_xacro_model/meshes/Suspension_6.STL"/>
           </geometry>
           <material name="">
@@ -751,5 +751,5 @@
           <origin rpy="0 0 0" xyz="0 0 0"/>
           <geometry>
-            <mesh filename="file://$(find j8_xacro_model)/meshes/Suspension_6.STL"/>
+            <mesh filename="package://j8_xacro_model/meshes/Suspension_6.STL"/>
           </geometry>
         </collision>
@@ -781,5 +781,5 @@
             <cylinder length="0.30" radius="0.298"/>
           </geometry>
-          <geometry> <mesh filename="file://$(find j8_xacro_model)/meshes/Wheel6.STL"/>
+          <geometry> <mesh filename="package://j8_xacro_model/meshes/Wheel6.STL"/>
             </geometry>
           <material name="">
@@ -793,5 +793,5 @@
           </geometry>
           <geometry>
-              <mesh filename="file://$(find j8_xacro_model)/meshes/Wheel6.STL"/>
+              <mesh filename="package://j8_xacro_model/meshes/Wheel6.STL"/>
             </geometry>
         </collision>
@@ -834,5 +834,5 @@
           <origin rpy="0 0 0" xyz="0 0 0"/>
           <geometry>
-            <mesh filename="file://$(find j8_xacro_model)/meshes/Suspension_7.STL"/>
+            <mesh filename="package://j8_xacro_model/meshes/Suspension_7.STL"/>
           </geometry>
           <material name="">
@@ -843,5 +843,5 @@
           <origin rpy="0 0 0" xyz="0 0 0"/>
           <geometry>
-            <mesh filename="file://$(find j8_xacro_model)/meshes/Suspension_7.STL"/>
+            <mesh filename="package://j8_xacro_model/meshes/Suspension_7.STL"/>
           </geometry>
         </collision>
@@ -873,5 +873,5 @@
             <cylinder length="0.30" radius="0.298"/>
           </geometry>
-          <geometry> <mesh filename="file://$(find j8_xacro_model)/meshes/Wheel7.STL"/>
+          <geometry> <mesh filename="package://j8_xacro_model/meshes/Wheel7.STL"/>
             </geometry>
           <material name="">
@@ -885,5 +885,5 @@
           </geometry>
           <geometry>
-              <mesh filename="file://$(find j8_xacro_model)/meshes/Wheel7.STL"/>
+              <mesh filename="package://j8_xacro_model/meshes/Wheel7.STL"/>
             </geometry>
         </collision>
@@ -926,5 +926,5 @@
           <origin rpy="0 0 0" xyz="0 0 0"/>
           <geometry>
-            <mesh filename="file://$(find j8_xacro_model)/meshes/Suspension_8.STL"/>
+            <mesh filename="package://j8_xacro_model/meshes/Suspension_8.STL"/>
           </geometry>
           <material name="">
@@ -935,5 +935,5 @@
           <origin rpy="0 0 0" xyz="0 0 0"/>
           <geometry>
-            <mesh filename="file://$(find j8_xacro_model)/meshes/Suspension_8.STL"/>
+            <mesh filename="package://j8_xacro_model/meshes/Suspension_8.STL"/>
           </geometry>
         </collision>
@@ -965,5 +965,5 @@
             <cylinder length="0.30" radius="0.298"/>
           </geometry>
-          <geometry> <mesh filename="file://$(find j8_xacro_model)/meshes/Wheel8.STL"/>
+          <geometry> <mesh filename="package://j8_xacro_model/meshes/Wheel8.STL"/>
             </geometry>
           <material name="">
@@ -977,5 +977,5 @@
           </geometry>
           <geometry>
-              <mesh filename="file://$(find j8_xacro_model)/meshes/wWheel8.STL"/>
+              <mesh filename="package://j8_xacro_model/meshes/wWheel8.STL"/>
             </geometry>
         </collision>

File: src/gazebo_sim_pkgs/j8_xacro_model/urdf/camera.xacro (robot description, xacro)
@@ -11,5 +11,5 @@
         <origin xyz="0 0 0" rpy="0 0 0" />
         <geometry>
-          <mesh filename="file://$(find j8_xacro_model)/meshes/Back_camera.STL" />
+          <mesh filename="package://j8_xacro_model/meshes/Back_camera.STL" />
         </geometry>
         <!-- The color is predefined -->
@@ -21,5 +21,5 @@
         <origin xyz="0 0 0" rpy="0 0 0" />
         <geometry>
-          <mesh filename="file://$(find j8_xacro_model)/meshes/Back_camera.STL" />
+          <mesh filename="package://j8_xacro_model/meshes/Back_camera.STL" />
         </geometry>
       </collision>

File: src/gazebo_sim_pkgs/j8_xacro_model/urdf/fixposition_holder.xacro (robot description, xacro)
@@ -25,5 +25,5 @@
       <geometry>
         <mesh
-          filename="file://$(find j8_xacro_model)/meshes/Fixposion_base.STL" />
+          filename="package://j8_xacro_model/meshes/Fixposion_base.STL" />
       </geometry>
       <material
@@ -39,5 +39,5 @@
       <geometry>
         <mesh
-          filename="file://$(find j8_xacro_model)/meshes/Fixposion_base.STL" />
+          filename="package://j8_xacro_model/meshes/Fixposion_base.STL" />
       </geometry>
     </collision>
@@ -77,5 +77,5 @@
       <geometry>
         <mesh
-          filename="file://$(find j8_xacro_model)/meshes/Left_fixposition_feet.STL" />
+          filename="package://j8_xacro_model/meshes/Left_fixposition_feet.STL" />
       </geometry>
       <material
@@ -91,5 +91,5 @@
       <geometry>
         <mesh
-          filename="file://$(find j8_xacro_model)/meshes/Left_fixposition_feet.STL" />
+          filename="package://j8_xacro_model/meshes/Left_fixposition_feet.STL" />
       </geometry>
     </collision>
@@ -131,5 +131,5 @@
       <geometry>
         <mesh
-          filename="file://$(find j8_xacro_model)/meshes/Left_fixposition_holder.STL" />
+          filename="package://j8_xacro_model/meshes/Left_fixposition_holder.STL" />
       </geometry>
       <material
@@ -145,5 +145,5 @@
       <geometry>
         <mesh
-          filename="file://$(find j8_xacro_model)/meshes/Left_fixposition_holder.STL" />
+          filename="package://j8_xacro_model/meshes/Left_fixposition_holder.STL" />
       </geometry>
     </collision>
@@ -185,5 +185,5 @@
       <geometry>
         <mesh
-          filename="file://$(find j8_xacro_model)/meshes/Central_fixposition_feet.STL" />
+          filename="package://j8_xacro_model/meshes/Central_fixposition_feet.STL" />
       </geometry>
       <material
@@ -199,5 +199,5 @@
       <geometry>
         <mesh
-          filename="file://$(find j8_xacro_model)/meshes/Central_fixposition_feet.STL" />
+          filename="package://j8_xacro_model/meshes/Central_fixposition_feet.STL" />
       </geometry>
     </collision>
@@ -239,5 +239,5 @@
       <geometry>
         <mesh
-          filename="file://$(find j8_xacro_model)/meshes/Central_fixposition_holder.STL" />
+          filename="package://j8_xacro_model/meshes/Central_fixposition_holder.STL" />
       </geometry>
       <material
@@ -253,5 +253,5 @@
       <geometry>
         <mesh
-          filename="file://$(find j8_xacro_model)/meshes/Central_fixposition_holder.STL" />
+          filename="package://j8_xacro_model/meshes/Central_fixposition_holder.STL" />
       </geometry>
     </collision>
@@ -293,5 +293,5 @@
       <geometry>
         <mesh
-          filename="file://$(find j8_xacro_model)/meshes/Right_fixposition_feet.STL" />
+          filename="package://j8_xacro_model/meshes/Right_fixposition_feet.STL" />
       </geometry>
       <material
@@ -307,5 +307,5 @@
       <geometry>
         <mesh
-          filename="file://$(find j8_xacro_model)/meshes/Right_fixposition_feet.STL" />
+          filename="package://j8_xacro_model/meshes/Right_fixposition_feet.STL" />
       </geometry>
     </collision>
@@ -347,5 +347,5 @@
       <geometry>
         <mesh
-          filename="file://$(find j8_xacro_model)/meshes/Right_fixposition_holder.STL" />
+          filename="package://j8_xacro_model/meshes/Right_fixposition_holder.STL" />
       </geometry>
       <material
@@ -361,5 +361,5 @@
       <geometry>
         <mesh
-          filename="file://$(find j8_xacro_model)/meshes/Right_fixposition_holder.STL" />
+          filename="package://j8_xacro_model/meshes/Right_fixposition_holder.STL" />
       </geometry>
     </collision>

File: src/gazebo_sim_pkgs/j8_xacro_model/urdf/fixposition_sensor.xacro (robot description, xacro)
@@ -12,5 +12,5 @@
         <origin xyz="0 0 0" rpy="0 0 0" />
         <geometry>
-          <mesh filename="file://$(find j8_xacro_model)/meshes/Fix_position_metal_frame.STL" />
+          <mesh filename="package://j8_xacro_model/meshes/Fix_position_metal_frame.STL" />
         </geometry>
         <material name="">
@@ -21,5 +21,5 @@
         <origin xyz="0 0 0" rpy="0 0 0" />
         <geometry>
-          <mesh filename="file://$(find j8_xacro_model)/meshes/Fix_position_metal_frame.STL" />
+          <mesh filename="package://j8_xacro_model/meshes/Fix_position_metal_frame.STL" />
         </geometry>
       </collision>
@@ -43,5 +43,5 @@
         <origin xyz="0 0 0" rpy="0 0 0" />
         <geometry>
-          <mesh filename="file://$(find j8_xacro_model)/meshes/Fix_position_left_antenna.STL" />
+          <mesh filename="package://j8_xacro_model/meshes/Fix_position_left_antenna.STL" />
         </geometry>
         <material name="">
@@ -52,5 +52,5 @@
         <origin xyz="0 0 0" rpy="0 0 0" />
         <geometry>
-          <mesh filename="file://$(find j8_xacro_model)/meshes/Fix_position_left_antenna.STL" />
+          <mesh filename="package://j8_xacro_model/meshes/Fix_position_left_antenna.STL" />
         </geometry>
       </collision>
@@ -73,5 +73,5 @@
         <origin xyz="0 0 0" rpy="0 0 0" />
         <geometry>
-          <mesh filename="file://$(find j8_xacro_model)/meshes/Fixposition_right_antenna.STL" />
+          <mesh filename="package://j8_xacro_model/meshes/Fixposition_right_antenna.STL" />
         </geometry>
         <material name="">
@@ -82,5 +82,5 @@
         <origin xyz="0 0 0" rpy="0 0 0" />
         <geometry>
-          <mesh filename="file://$(find j8_xacro_model)/meshes/Fixposition_right_antenna.STL" />
+          <mesh filename="package://j8_xacro_model/meshes/Fixposition_right_antenna.STL" />
         </geometry>
       </collision>
@@ -103,5 +103,5 @@
         <origin xyz="0 0 0" rpy="0 0 0" />
         <geometry>
-          <mesh filename="file://$(find j8_xacro_model)/meshes/Fixposition_lower_case.STL" />
+          <mesh filename="package://j8_xacro_model/meshes/Fixposition_lower_case.STL" />
         </geometry>
         <material name="">
@@ -112,5 +112,5 @@
         <origin xyz="0 0 0" rpy="0 0 0" />
         <geometry>
-          <mesh filename="file://$(find j8_xacro_model)/meshes/Fixposition_lower_case.STL" />
+          <mesh filename="package://j8_xacro_model/meshes/Fixposition_lower_case.STL" />
         </geometry>
       </collision>
@@ -133,5 +133,5 @@
         <origin xyz="0 0 0" rpy="0 0 0" />
         <geometry>
-          <mesh filename="file://$(find j8_xacro_model)/meshes/Fixposition_upper_case.STL" />
+          <mesh filename="package://j8_xacro_model/meshes/Fixposition_upper_case.STL" />
         </geometry>
         <material name="">
@@ -142,5 +142,5 @@
         <origin xyz="0 0 0" rpy="0 0 0" />
         <geometry>
-          <mesh filename="file://$(find j8_xacro_model)/meshes/Fixposition_upper_case.STL" />
+          <mesh filename="package://j8_xacro_model/meshes/Fixposition_upper_case.STL" />
         </geometry>
       </collision>
@@ -163,5 +163,5 @@
         <origin xyz="0 0 0" rpy="0 0 0" />
         <geometry>
-          <mesh filename="file://$(find j8_xacro_model)/meshes/Fixposition_camera.STL" />
+          <mesh filename="package://j8_xacro_model/meshes/Fixposition_camera.STL" />
         </geometry>
         <material name="">
@@ -172,5 +172,5 @@
         <origin xyz="0 0 0" rpy="0 0 0" />
         <geometry>
-          <mesh filename="file://$(find j8_xacro_model)/meshes/Fixposition_camera.STL" />
+          <mesh filename="package://j8_xacro_model/meshes/Fixposition_camera.STL" />
         </geometry>
       </collision>

File: src/gazebo_sim_pkgs/j8_xacro_model/urdf/gps.xacro (robot description, xacro)
@@ -27,5 +27,5 @@
       <geometry>
         <mesh
-          filename="file://$(find j8_xacro_model)/meshes/Left_gps.STL" />
+          filename="package://j8_xacro_model/meshes/Left_gps.STL" />
       </geometry>
       <material
@@ -41,5 +41,5 @@
       <geometry>
         <mesh
-          filename="file://$(find j8_xacro_model)/meshes/Left_gps.STL" />
+          filename="package://j8_xacro_model/meshes/Left_gps.STL" />
       </geometry>
     </collision>

File: src/gazebo_sim_pkgs/j8_xacro_model/urdf/gps_holder.xacro (robot description, xacro)
@@ -11,5 +11,5 @@
         <origin xyz="0 0 0" rpy="0 0 0" />
         <geometry>
-          <mesh filename="file://$(find j8_xacro_model)/meshes/Right_gps_holder.STL" />
+          <mesh filename="package://j8_xacro_model/meshes/Right_gps_holder.STL" />
         </geometry>
         <material name="">
@@ -20,5 +20,5 @@
         <origin xyz="0 0 0" rpy="0 0 0" />
         <geometry>
-          <mesh filename="file://$(find j8_xacro_model)/meshes/Right_gps_holder.STL" />
+          <mesh filename="package://j8_xacro_model/meshes/Right_gps_holder.STL" />
         </geometry>
       </collision>

File: src/gazebo_sim_pkgs/j8_xacro_model/urdf/panel.xacro (robot description, xacro)
@@ -11,5 +11,5 @@
         <origin xyz="0 0 0" rpy="0 0 0"/>
         <geometry>
-          <mesh filename="file://$(find j8_xacro_model)/meshes/${name}.STL"/>
+          <mesh filename="package://j8_xacro_model/meshes/${name}.STL"/>
         </geometry>
         <material name="">
@@ -20,5 +20,5 @@
         <origin xyz="0 0 0" rpy="0 0 0"/>
         <geometry>
-          <mesh filename="file://$(find j8_xacro_model)/meshes/${name}.STL"/>
+          <mesh filename="package://j8_xacro_model/meshes/${name}.STL"/>
         </geometry>
       </collision>
