Commit message: update the code

File: src/gazebo_sim_pkgs/j8_xacro_model/urdf/side_bar.xacro (robot description, xacro)
@@ -13,5 +13,5 @@
         <origin xyz="0 0 0" rpy="0 0 0" />
         <geometry>
-          <mesh filename="file://$(find j8_xacro_model)/meshes/${name}.STL" />
+          <mesh filename="package://j8_xacro_model/meshes/${name}.STL" />
         </geometry>
         <!-- The color is defined in the main file or through a gazebo tag -->
@@ -20,5 +20,5 @@
         <origin xyz="0 0 0" rpy="0 0 0" />
         <geometry>
-          <mesh filename="file://$(find j8_xacro_model)/meshes/${name}.STL" />
+          <mesh filename="package://j8_xacro_model/meshes/${name}.STL" />
         </geometry>
       </collision>

Commit message: first commit

File: src/gazebo_sim_pkgs/j8_xacro_model/urdf/argo_j8.xacro (robot description, xacro)
@@ -43,5 +43,5 @@
       <geometry>
         <mesh
-          filename="package://j8_xacro_model/meshes/base_link.STL" />
+          filename="file://$(find j8_xacro_model)/meshes/base_link.STL" />
       </geometry>
       <material
@@ -57,5 +57,5 @@
       <geometry>
         <mesh
-          filename="package://j8_xacro_model/meshes/base_link.STL" />
+          filename="file://$(find j8_xacro_model)/meshes/base_link.STL" />
       </geometry>
     </collision>
@@ -85,5 +85,5 @@
       <geometry>
         <mesh
-          filename="package://j8_xacro_model/meshes/J8_top.STL" />
+          filename="file://$(find j8_xacro_model)/meshes/J8_top.STL" />
       </geometry>
       <material
@@ -99,5 +99,5 @@
       <geometry>
         <mesh
-          filename="package://j8_xacro_model/meshes/J8_top.STL" />
+          filename="file://$(find j8_xacro_model)/meshes/J8_top.STL" />
       </geometry>
     </collision>
@@ -139,5 +139,5 @@
       <geometry>
         <mesh
-          filename="package://j8_xacro_model/meshes/Bridge.STL" />
+          filename="file://$(find j8_xacro_model)/meshes/Bridge.STL" />
       </geometry>
       <material
@@ -153,5 +153,5 @@
       <geometry>
         <mesh
-          filename="package://j8_xacro_model/meshes/Bridge.STL" />
+          filename="file://$(find j8_xacro_model)/meshes/Bridge.STL" />
       </geometry>
     </collision>
@@ -196,5 +196,5 @@
             <origin rpy="0 0 0" xyz="0 0 0"/>
             <geometry>
-              <mesh filename="package://j8_xacro_model/meshes/Sick.STL"/>
+              <mesh filename="file://$(find j8_xacro_model)/meshes/Sick.STL"/>
             </geometry>
             <!-- Default color for all lidars -->
@@ -206,5 +206,5 @@
             <origin rpy="0 0 0" xyz="0 0 0"/>
             <geometry>
-              <mesh filename="package://j8_xacro_model/meshes/Sick.STL"/>
+              <mesh filename="file://$(find j8_xacro_model)/meshes/Sick.STL"/>
             </geometry>
           </collision>
@@ -227,5 +227,5 @@
       <origin rpy="0 0 0" xyz="0 0 0"/>
       <geometry>
-        <mesh filename="package://j8_xacro_model/meshes/Velodyne.STL"/>
+        <mesh filename="file://$(find j8_xacro_model)/meshes/Velodyne.STL"/>
       </geometry>
       <!-- Default color for all lidars -->
@@ -237,11 +237,11 @@
       <origin rpy="0 0 0" xyz="0 0 0"/>
       <geometry>
-        <mesh filename="package://j8_xacro_model/meshes/Velodyne.STL"/>
+        <mesh filename="file://$(find j8_xacro_model)/meshes/Velodyne.STL"/>
       </geometry>
     </collision>
   </link>
   <joint name="Velodyne_joint" type="fixed">
-    <origin rpy="0 0 0" xyz="0.93 0.0 1.0"/>
-    <parent link="J8_top"/>
+    <origin rpy="0 0 0" xyz="0.8026628 0.0075201 0.96892"/>
+    <parent link="base_link"/>
     <child link="Velodyne_link"/>
     <axis xyz="0 0 0"/>
@@ -282,5 +282,5 @@
           <origin rpy="0 0 0" xyz="0 0 0"/>
           <geometry>
-            <mesh filename="package://j8_xacro_model/meshes/Suspension_1.STL"/>
+            <mesh filename="file://$(find j8_xacro_model)/meshes/Suspension_1.STL"/>
           </geometry>
           <material name="">
@@ -291,5 +291,5 @@
           <origin rpy="0 0 0" xyz="0 0 0"/>
           <geometry>
-            <mesh filename="package://j8_xacro_model/meshes/Suspension_1.STL"/>
+            <mesh filename="file://$(find j8_xacro_model)/meshes/Suspension_1.STL"/>
           </geometry>
         </collision>
@@ -321,5 +321,5 @@
             <cylinder length="0.30" radius="0.298"/>
           </geometry>
-          <geometry> <mesh filename="package://j8_xacro_model/meshes/Wheel1.STL"/>
+          <geometry> <mesh filename="file://$(find j8_xacro_model)/meshes/Wheel1.STL"/>
             </geometry>
           <material name="">
@@ -333,5 +333,5 @@
           </geometry>
           <geometry>
-              <mesh filename="package://j8_xacro_model/meshes/Wheel1.STL"/>
+              <mesh filename="file://$(find j8_xacro_model)/meshes/Wheel1.STL"/>
             </geometry>
         </collision>
@@ -374,5 +374,5 @@
           <origin rpy="0 0 0" xyz="0 0 0"/>
           <geometry>
-            <mesh filename="package://j8_xacro_model/meshes/Suspension_2.STL"/>
+            <mesh filename="file://$(find j8_xacro_model)/meshes/Suspension_2.STL"/>
           </geometry>
           <material name="">
@@ -383,5 +383,5 @@
           <origin rpy="0 0 0" xyz="0 0 0"/>
           <geometry>
-            <mesh filename="package://j8_xacro_model/meshes/Suspension_2.STL"/>
+            <mesh filename="file://$(find j8_xacro_model)/meshes/Suspension_2.STL"/>
           </geometry>
         </collision>
@@ -413,5 +413,5 @@
             <cylinder length="0.30" radius="0.298"/>
           </geometry>
-          <geometry> <mesh filename="package://j8_xacro_model/meshes/Wheel2.STL"/>
+          <geometry> <mesh filename="file://$(find j8_xacro_model)/meshes/Wheel2.STL"/>
             </geometry>
           <material name="">
@@ -425,5 +425,5 @@
           </geometry>
           <geometry>
-              <mesh filename="package://j8_xacro_model/meshes/Wheel2.STL"/>
+              <mesh filename="file://$(find j8_xacro_model)/meshes/Wheel2.STL"/>
             </geometry>
         </collision>
@@ -466,5 +466,5 @@
           <origin rpy="0 0 0" xyz="0 0 0"/>
           <geometry>
-            <mesh filename="package://j8_xacro_model/meshes/Suspension_3.STL"/>
+            <mesh filename="file://$(find j8_xacro_model)/meshes/Suspension_3.STL"/>
           </geometry>
           <material name="">
@@ -475,5 +475,5 @@
           <origin rpy="0 0 0" xyz="0 0 0"/>
           <geometry>
-            <mesh filename="package://j8_xacro_model/meshes/Suspension_3.STL"/>
+            <mesh filename="file://$(find j8_xacro_model)/meshes/Suspension_3.STL"/>
           </geometry>
         </collision>
@@ -505,5 +505,5 @@
             <cylinder length="0.30" radius="0.298"/>
           </geometry>
-          <geometry> <mesh filename="package://j8_xacro_model/meshes/Wheel3.STL"/>
+          <geometry> <mesh filename="file://$(find j8_xacro_model)/meshes/Wheel3.STL"/>
             </geometry>
           <material name="">
@@ -517,5 +517,5 @@
           </geometry>
           <geometry>
-              <mesh filename="package://j8_xacro_model/meshes/Wheel3.STL"/>
+              <mesh filename="file://$(find j8_xacro_model)/meshes/Wheel3.STL"/>
             </geometry>
         </collision>
@@ -558,5 +558,5 @@
           <origin rpy="0 0 0" xyz="0 0 0"/>
           <geometry>
-            <mesh filename="package://j8_xacro_model/meshes/Suspension_4.STL"/>
+            <mesh filename="file://$(find j8_xacro_model)/meshes/Suspension_4.STL"/>
           </geometry>
           <material name="">
@@ -567,5 +567,5 @@
           <origin rpy="0 0 0" xyz="0 0 0"/>
           <geometry>
-            <mesh filename="package://j8_xacro_model/meshes/Suspension_4.STL"/>
+            <mesh filename="file://$(find j8_xacro_model)/meshes/Suspension_4.STL"/>
           </geometry>
         </collision>
@@ -597,5 +597,5 @@
             <cylinder length="0.30" radius="0.298"/>
           </geometry>
-          <geometry> <mesh filename="package://j8_xacro_model/meshes/Wheel4.STL"/>
+          <geometry> <mesh filename="file://$(find j8_xacro_model)/meshes/Wheel4.STL"/>
             </geometry>
           <material name="">
@@ -609,5 +609,5 @@
           </geometry>
           <geometry>
-              <mesh filename="package://j8_xacro_model/meshes/Wheel4.STL"/>
+              <mesh filename="file://$(find j8_xacro_model)/meshes/Wheel4.STL"/>
             </geometry>
         </collision>
@@ -650,5 +650,5 @@
           <origin rpy="0 0 0" xyz="0 0 0"/>
           <geometry>
-            <mesh filename="package://j8_xacro_model/meshes/Suspension_5.STL"/>
+            <mesh filename="file://$(find j8_xacro_model)/meshes/Suspension_5.STL"/>
           </geometry>
           <material name="">
@@ -659,5 +659,5 @@
           <origin rpy="0 0 0" xyz="0 0 0"/>
           <geometry>
-            <mesh filename="package://j8_xacro_model/meshes/Suspension_5.STL"/>
+            <mesh filename="file://$(find j8_xacro_model)/meshes/Suspension_5.STL"/>
           </geometry>
         </collision>
@@ -689,5 +689,5 @@
             <cylinder length="0.30" radius="0.298"/>
           </geometry>
-          <geometry> <mesh filename="package://j8_xacro_model/meshes/Wheel5.STL"/>
+          <geometry> <mesh filename="file://$(find j8_xacro_model)/meshes/Wheel5.STL"/>
             </geometry>
           <material name="">
@@ -701,5 +701,5 @@
           </geometry>
           <geometry>
-              <mesh filename="package://j8_xacro_model/meshes/Wheel5.STL"/>
+              <mesh filename="file://$(find j8_xacro_model)/meshes/Wheel5.STL"/>
             </geometry>
         </collision>
@@ -742,5 +742,5 @@
           <origin rpy="0 0 0" xyz="0 0 0"/>
           <geometry>
-            <mesh filename="package://j8_xacro_model/meshes/Suspension_6.STL"/>
+            <mesh filename="file://$(find j8_xacro_model)/meshes/Suspension_6.STL"/>
           </geometry>
           <material name="">
@@ -751,5 +751,5 @@
           <origin rpy="0 0 0" xyz="0 0 0"/>
           <geometry>
-            <mesh filename="package://j8_xacro_model/meshes/Suspension_6.STL"/>
+            <mesh filename="file://$(find j8_xacro_model)/meshes/Suspension_6.STL"/>
           </geometry>
         </collision>
@@ -781,5 +781,5 @@
             <cylinder length="0.30" radius="0.298"/>
           </geometry>
-          <geometry> <mesh filename="package://j8_xacro_model/meshes/Wheel6.STL"/>
+          <geometry> <mesh filename="file://$(find j8_xacro_model)/meshes/Wheel6.STL"/>
             </geometry>
           <material name="">
@@ -793,5 +793,5 @@
           </geometry>
           <geometry>
-              <mesh filename="package://j8_xacro_model/meshes/Wheel6.STL"/>
+              <mesh filename="file://$(find j8_xacro_model)/meshes/Wheel6.STL"/>
             </geometry>
         </collision>
@@ -834,5 +834,5 @@
           <origin rpy="0 0 0" xyz="0 0 0"/>
           <geometry>
-            <mesh filename="package://j8_xacro_model/meshes/Suspension_7.STL"/>
+            <mesh filename="file://$(find j8_xacro_model)/meshes/Suspension_7.STL"/>
           </geometry>
           <material name="">
@@ -843,5 +843,5 @@
           <origin rpy="0 0 0" xyz="0 0 0"/>
           <geometry>
-            <mesh filename="package://j8_xacro_model/meshes/Suspension_7.STL"/>
+            <mesh filename="file://$(find j8_xacro_model)/meshes/Suspension_7.STL"/>
           </geometry>
         </collision>
@@ -873,5 +873,5 @@
             <cylinder length="0.30" radius="0.298"/>
           </geometry>
-          <geometry> <mesh filename="package://j8_xacro_model/meshes/Wheel7.STL"/>
+          <geometry> <mesh filename="file://$(find j8_xacro_model)/meshes/Wheel7.STL"/>
             </geometry>
           <material name="">
@@ -885,5 +885,5 @@
           </geometry>
           <geometry>
-              <mesh filename="package://j8_xacro_model/meshes/Wheel7.STL"/>
+              <mesh filename="file://$(find j8_xacro_model)/meshes/Wheel7.STL"/>
             </geometry>
         </collision>
@@ -926,5 +926,5 @@
           <origin rpy="0 0 0" xyz="0 0 0"/>
           <geometry>
-            <mesh filename="package://j8_xacro_model/meshes/Suspension_8.STL"/>
+            <mesh filename="file://$(find j8_xacro_model)/meshes/Suspension_8.STL"/>
           </geometry>
           <material name="">
@@ -935,5 +935,5 @@
           <origin rpy="0 0 0" xyz="0 0 0"/>
           <geometry>
-            <mesh filename="package://j8_xacro_model/meshes/Suspension_8.STL"/>
+            <mesh filename="file://$(find j8_xacro_model)/meshes/Suspension_8.STL"/>
           </geometry>
         </collision>
@@ -965,5 +965,5 @@
             <cylinder length="0.30" radius="0.298"/>
           </geometry>
-          <geometry> <mesh filename="package://j8_xacro_model/meshes/Wheel8.STL"/>
+          <geometry> <mesh filename="file://$(find j8_xacro_model)/meshes/Wheel8.STL"/>
             </geometry>
           <material name="">
@@ -977,5 +977,5 @@
           </geometry>
           <geometry>
-              <mesh filename="package://j8_xacro_model/meshes/wWheel8.STL"/>
+              <mesh filename="file://$(find j8_xacro_model)/meshes/wWheel8.STL"/>
             </geometry>
         </collision>
@@ -1011,5 +1011,5 @@
 <xacro:bridge_joint xyz="-0.0028148 -0.11697 0.21171" rpy="1.5708 0 1.5708"/>-->
 <!-- Fixposition sensor-->
-  <xacro:fixposition_full_setup parent="Bridge" xyz="-0.0028148 -0.11697 0.21171" rpy="1.5708 0 1.5708"/>
+  <xacro:fixposition_full_setup parent="Bridge" xyz="0.0094278 0.1804302 0.1437104" rpy="1.5708 0 1.5708"/>
  <gazebo>
   <!-- Diff drive plugin configuration -->

File: src/gazebo_sim_pkgs/j8_xacro_model/urdf/fixposition_sensor.xacro (robot description, xacro)
@@ -12,5 +12,5 @@
         <origin xyz="0 0 0" rpy="0 0 0" />
         <geometry>
-          <mesh filename="package://j8_xacro_model/meshes/Fix_position_metal_frame.STL" />
+          <mesh filename="file://$(find j8_xacro_model)/meshes/Fix_position_metal_frame.STL" />
         </geometry>
         <material name="">
@@ -21,5 +21,5 @@
         <origin xyz="0 0 0" rpy="0 0 0" />
         <geometry>
-          <mesh filename="package://j8_xacro_model/meshes/Fix_position_metal_frame.STL" />
+          <mesh filename="file://$(find j8_xacro_model)/meshes/Fix_position_metal_frame.STL" />
         </geometry>
       </collision>
@@ -43,5 +43,5 @@
         <origin xyz="0 0 0" rpy="0 0 0" />
         <geometry>
-          <mesh filename="package://j8_xacro_model/meshes/Fix_position_left_antenna.STL" />
+          <mesh filename="file://$(find j8_xacro_model)/meshes/Fix_position_left_antenna.STL" />
         </geometry>
         <material name="">
@@ -52,5 +52,5 @@
         <origin xyz="0 0 0" rpy="0 0 0" />
         <geometry>
-          <mesh filename="package://j8_xacro_model/meshes/Fix_position_left_antenna.STL" />
+          <mesh filename="file://$(find j8_xacro_model)/meshes/Fix_position_left_antenna.STL" />
         </geometry>
       </collision>
@@ -73,5 +73,5 @@
         <origin xyz="0 0 0" rpy="0 0 0" />
         <geometry>
-          <mesh filename="package://j8_xacro_model/meshes/Fixposition_right_antenna.STL" />
+          <mesh filename="file://$(find j8_xacro_model)/meshes/Fixposition_right_antenna.STL" />
         </geometry>
         <material name="">
@@ -82,5 +82,5 @@
         <origin xyz="0 0 0" rpy="0 0 0" />
         <geometry>
-          <mesh filename="package://j8_xacro_model/meshes/Fixposition_right_antenna.STL" />
+          <mesh filename="file://$(find j8_xacro_model)/meshes/Fixposition_right_antenna.STL" />
         </geometry>
       </collision>
@@ -103,5 +103,5 @@
         <origin xyz="0 0 0" rpy="0 0 0" />
         <geometry>
-          <mesh filename="package://j8_xacro_model/meshes/Fixposition_lower_case.STL" />
+          <mesh filename="file://$(find j8_xacro_model)/meshes/Fixposition_lower_case.STL" />
         </geometry>
         <material name="">
@@ -112,5 +112,5 @@
         <origin xyz="0 0 0" rpy="0 0 0" />
         <geometry>
-          <mesh filename="package://j8_xacro_model/meshes/Fixposition_lower_case.STL" />
+          <mesh filename="file://$(find j8_xacro_model)/meshes/Fixposition_lower_case.STL" />
         </geometry>
       </collision>
@@ -133,5 +133,5 @@
         <origin xyz="0 0 0" rpy="0 0 0" />
         <geometry>
-          <mesh filename="package://j8_xacro_model/meshes/Fixposition_upper_case.STL" />
+          <mesh filename="file://$(find j8_xacro_model)/meshes/Fixposition_upper_case.STL" />
         </geometry>
         <material name="">
@@ -142,5 +142,5 @@
         <origin xyz="0 0 0" rpy="0 0 0" />
         <geometry>
-          <mesh filename="package://j8_xacro_model/meshes/Fixposition_upper_case.STL" />
+          <mesh filename="file://$(find j8_xacro_model)/meshes/Fixposition_upper_case.STL" />
         </geometry>
       </collision>
@@ -163,5 +163,5 @@
         <origin xyz="0 0 0" rpy="0 0 0" />
         <geometry>
-          <mesh filename="package://j8_xacro_model/meshes/Fixposition_camera.STL" />
+          <mesh filename="file://$(find j8_xacro_model)/meshes/Fixposition_camera.STL" />
         </geometry>
         <material name="">
@@ -172,5 +172,5 @@
         <origin xyz="0 0 0" rpy="0 0 0" />
         <geometry>
-          <mesh filename="package://j8_xacro_model/meshes/Fixposition_camera.STL" />
+          <mesh filename="file://$(find j8_xacro_model)/meshes/Fixposition_camera.STL" />
         </geometry>
       </collision>
