Commit message: update j8

File: src/gazebo_sim_pkgs/j8_xacro_model/urdf/argo_j8.xacro (robot description, xacro)
@@ -242,5 +242,5 @@
   </link>
   <joint name="Velodyne_joint" type="fixed">
-    <origin rpy="0 0 0" xyz="0.8026628 0.0075201 0.96892"/>
+    <origin rpy="0 0 -1.5707963267948966" xyz="0.8026628 0.0075201 0.96892"/>
     <parent link="base_link"/>
     <child link="Velodyne_link"/>

Commit message: news features for dem fucntion and compress map, fix a few things and bugs

File: src/gazebo_sim_pkgs/j8_xacro_model/urdf/argo_j8.xacro (robot description, xacro)
@@ -242,5 +242,5 @@
   </link>
   <joint name="Velodyne_joint" type="fixed">
-    <origin rpy="0 0 -1.5707963267948966" xyz="0.8026628 0.0075201 0.96892"/>
+    <origin rpy="0 0 0" xyz="0.8026628 0.0075201 0.96892"/>
     <parent link="base_link"/>
     <child link="Velodyne_link"/>
